File: rp2350-v0.2/rp2350-v0.2/accel_bma400.kicad_sch (KiCad schematic)
At the start: 4 parts

Commit message: v0.2: schematic draft 1 done
Parts:
- JP3: footprint (none) -> CustomFootprints:BridgedJumper_P2.54mm
Changed lines of the file:
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@@
 			)
 		)
-		(property "Footprint" ""
+		(property "Footprint" "CustomFootprints:BridgedJumper_P2.54mm"
 			(at 189.23 59.69 0)
 			(effects
