File: rp2350-v0.2/rp2350-v0.2/eeprom_m95512.kicad_sch (KiCad schematic)
At the start: 5 parts, among them IC1 M95512-RMN6TP

Commit message: v0.2: schematic draft 1 done
Parts:
- IC1: footprint (none) -> SamacSys_Parts:SOIC127P600X175-8N
- JP1: footprint (none) -> CustomFootprints:BridgedJumper_P2.54mm
Changed lines of the file:
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@@
 			)
 		)
-		(property "Footprint" ""
+		(property "Footprint" "SamacSys_Parts:SOIC127P600X175-8N"
 			(at 147.32 174.93 0)
 			(effects
@@
 			)
 		)
-		(property "Footprint" ""
+		(property "Footprint" "CustomFootprints:BridgedJumper_P2.54mm"
 			(at 179.07 57.15 0)
 			(effects
