File: rp2350-v0.2/rp2350-v0.2/flash_w25q1282.kicad_sch (KiCad schematic)
At the start: 4 parts, among them IC5 W25Q128JVSIM_TR

Commit message: v0.2: schematic draft 1 done
Parts:
- JP7: footprint (none) -> CustomFootprints:BridgedJumper_P2.54mm
Changed lines of the file:
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@@
 			)
 		)
-		(property "Footprint" ""
+		(property "Footprint" "CustomFootprints:BridgedJumper_P2.54mm"
 			(at 226.06 105.41 0)
 			(effects
