File: rp2350-v0.2/rp2350-v0.2/buttons_debounce.kicad_sch (KiCad schematic)
At the start: 12 parts, among them SW1 BUT_R, SW2 BUT_M, SW3 BUT_L

Commit message: v0.2: more progress on routing, nearly done
Parts:
- R12: footprint Capacitor_SMD:C_0402_1005Metric -> Resistor_SMD:R_0402_1005Metric
Changed lines of the file:
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@@
 			)
 		)
-		(property "Footprint" "Capacitor_SMD:C_0402_1005Metric"
+		(property "Footprint" "Resistor_SMD:R_0402_1005Metric"
 			(at 77.47 51.562 90)
 			(effects
