File: rp2350-v0.2/rp2350-v0.2/irda_pio.kicad_sch (KiCad schematic)
At the start: 6 parts, among them IC2 TFBS4711-TT1

Commit message: v0.2: schematic draft 1 done
Parts:
- JP2: footprint (none) -> CustomFootprints:BridgedJumper_P2.54mm
Changed lines of the file:
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@@
 			)
 		)
-		(property "Footprint" ""
+		(property "Footprint" "CustomFootprints:BridgedJumper_P2.54mm"
 			(at 167.64 81.28 0)
 			(effects

Commit message: v0.2: final big checks done, fixed IrDA footprint
Parts:
- IC2: footprint SamacSys_Parts:TFBS4711TT1 -> CustomFootprints:TFBS4711-TR
Changed lines of the file:
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@@
 			)
 		)
-		(property "Footprint" "SamacSys_Parts:TFBS4711TT1"
+		(property "Footprint" "CustomFootprints:TFBS4711-TR"
 			(at 83.82 195.25 0)
 			(effects
