File: rp2350-v0.2/rp2350-v0.2/sound_pwm.kicad_sch (KiCad schematic)
At the start: 1 part, among them J6 SPEAKER_CONNECTOR

Commit message: v0.2: update battery connector and labels
Parts:
- J6: footprint Resistor_SMD:R_0805_2012Metric -> Connector_PinHeader_2.54mm:PinHeader_1x02_P2.54mm_Vertical
Changed lines of the file:
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@@
 			)
 		)
-		(property "Footprint" "Resistor_SMD:R_0805_2012Metric"
+		(property "Footprint" "Connector_PinHeader_2.54mm:PinHeader_1x02_P2.54mm_Vertical"
 			(at 118.11 76.2 0)
 			(effects
