File: v0.3/accel_bma400.kicad_sch (KiCad schematic)
At the start: 4 parts

Commit message: v0.3: lots of routing done
Parts:
- removed NT1: NetTie_2, symbol Device:NetTie_2
Connections:
- net ACCEL_3V3 is gone; now on net +3.3V: AC1.3 (VDDIO), AC1.7 (VDD), C4.1, C5.1
Changed lines of the file:
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@@
 	(wire
 		(pts
-			(xy 184.15 59.69) (xy 170.18 59.69)
+			(xy 170.18 59.69) (xy 204.47 59.69)
 		)
 		(stroke
@@
 		(pts
 			(xy 161.29 90.17) (xy 161.29 92.71)
-		)
-		(stroke
-			(width 0)
-			(type default)
-		)
-	)
-	(wire
-		(pts
-			(xy 194.31 59.69) (xy 204.47 59.69)
 		)
 		(stroke
@@
 					(unit 1)
 				)
-			)
-		)
-	)
-	(symbol
-		(lib_id "Device:NetTie_2")
-		(at 186.69 59.69 0)
-		(unit 1)
-		(exclude_from_sim no)
-		(in_bom no)
-		(on_board yes)
-		(dnp no)
-		(fields_autoplaced yes)
-		(property "Reference" "NT1"
-			(at 186.69 54.61 0)
-			(effects
-				(font
-					(size 1.27 1.27)
-				)
-			)
-		)
-		(property "Value" "NetTie_2"
-			(at 186.69 57.15 0)
-			(effects
-				(font
-					(size 1.27 1.27)
-				)
-			)
-		)
-		(property "Footprint" ""
-			(at 186.69 59.69 0)
-			(effects
-				(font
-					(size 1.27 1.27)
-				)
-				(hide yes)
-			)
-		)
-		(property "Datasheet" "~"
-			(at 186.69 59.69 0)
-			(effects
-				(font
-					(size 1.27 1.27)
-				)
-				(hide yes)
-			)
-		)
-		(property "Description" "Net tie, 2 pins"
-			(at 186.69 59.69 0)
-			(effects
-				(font
-					(size 1.27 1.27)
-				)
-				(hide yes)
-			)
-		)
-		(pin "2"
-		)
-		(pin "1"
-		)
-		(instances
-			(project ""
-				(path "/5cbb45d4-7f83-48dd-a53b-5c75c7d1d827/ffe530de-e393-4ac8-a471-7661cdea5c19"
-					(reference "NT1")
-					(unit 1)
-				)
