File: v0.3/buttons_debounce.kicad_sch (KiCad schematic)
At the start: 12 parts, among them SW1 BUT_R, SW2 BUT_M, SW3 BUT_L

Commit message: v0.3: lots of routing done
Parts:
- SW1, SW2, SW3: footprint Button_Switch_SMD:SW_SPST_Omron_B3FS-101xP -> CustomFootprints:Button_membrane_5mm
Changed lines of the file:
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@@
 			)
 		)
-		(property "Footprint" "Button_Switch_SMD:SW_SPST_Omron_B3FS-101xP"
+		(property "Footprint" "CustomFootprints:Button_membrane_5mm"
 			(at 52.07 140.97 0)
 			(effects
@@
 			)
 		)
-		(property "Footprint" "Button_Switch_SMD:SW_SPST_Omron_B3FS-101xP"
+		(property "Footprint" "CustomFootprints:Button_membrane_5mm"
 			(at 54.61 48.26 0)
 			(effects
@@
 			)
 		)
-		(property "Footprint" "Button_Switch_SMD:SW_SPST_Omron_B3FS-101xP"
+		(property "Footprint" "CustomFootprints:Button_membrane_5mm"
 			(at 53.34 96.52 0)
 			(effects
