File: v0.3/eeprom_m95512.kicad_sch (KiCad schematic)
At the start: 5 parts, among them IC1 M95512-RMN6TP

Commit message: v0.3: lots of routing done
Parts:
- removed NT7: NetTie_2, symbol Device:NetTie_2
Connections:
- net EEPROM_3V3 is gone; now on net +3.3V: C1.1, IC1.3 (~{W}), IC1.7 (~{HOLD}), IC1.8 (VCC), R3.1
Changed lines of the file:
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@@
 	(wire
 		(pts
-			(xy 163.83 57.15) (xy 173.99 57.15)
+			(xy 163.83 57.15) (xy 193.04 57.15)
 		)
 		(stroke
@@
 		(pts
 			(xy 153.67 85.09) (xy 153.67 91.44)
-		)
-		(stroke
-			(width 0)
-			(type default)
-		)
-	)
-	(wire
-		(pts
-			(xy 179.07 57.15) (xy 193.04 57.15)
 		)
 		(stroke
@@
 					(unit 1)
 				)
-			)
-		)
-	)
-	(symbol
-		(lib_id "Device:NetTie_2")
-		(at 176.53 57.15 0)
-		(unit 1)
-		(exclude_from_sim no)
-		(in_bom no)
-		(on_board yes)
-		(dnp no)
-		(fields_autoplaced yes)
-		(property "Reference" "NT7"
-			(at 176.53 52.07 0)
-			(effects
-				(font
-					(size 1.27 1.27)
-				)
-			)
-		)
-		(property "Value" "NetTie_2"
-			(at 176.53 54.61 0)
-			(effects
-				(font
-					(size 1.27 1.27)
-				)
-			)
-		)
-		(property "Footprint" ""
-			(at 176.53 57.15 0)
-			(effects
-				(font
-					(size 1.27 1.27)
-				)
-				(hide yes)
-			)
-		)
-		(property "Datasheet" "~"
-			(at 176.53 57.15 0)
-			(effects
-				(font
-					(size 1.27 1.27)
-				)
-				(hide yes)
-			)
-		)
-		(property "Description" "Net tie, 2 pins"
-			(at 176.53 57.15 0)
-			(effects
-				(font
-					(size 1.27 1.27)
-				)
-				(hide yes)
-			)
-		)
-		(pin "1"
-		)
-		(pin "2"
-		)
-		(instances
-			(project ""
-				(path "/5cbb45d4-7f83-48dd-a53b-5c75c7d1d827/9111d733-478b-42e1-91b4-54aa10bab058"
-					(reference "NT7")
-					(unit 1)
-				)
