File: v0.3/screen_dw0180fmst08.kicad_sch (KiCad schematic)
At the start: 6 parts, among them J4 DO0180FMST08

Commit message: v0.3: lots of routing done
Parts:
- removed NT5, NT6: NetTie_2, symbol Device:NetTie_2
Connections:
- net SCREEN_3V3 is gone; now on net +3.3V: C21.1, J4.17 (IM1), J4.24 (VCI), J4.26 (VDDIO)
- net SCREEN_VSYS is gone; now on net VSYS: C19.2, C20.1, J4.18 (VBAT), J4.20 (VBAT)
Changed lines of the file:
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@@
-	(wire
-		(pts
-			(xy 232.41 60.96) (xy 252.73 60.96)
-		)
-		(stroke
-			(width 0)
-			(type default)
-		)
-	)
 	(wire
 		(pts
@@
 	(wire
 		(pts
-			(xy 215.9 60.96) (xy 227.33 60.96)
+			(xy 215.9 60.96) (xy 252.73 60.96)
 		)
 		(stroke
@@
 	(wire
 		(pts
-			(xy 231.14 41.91) (xy 252.73 41.91)
-		)
-		(stroke
-			(width 0)
-			(type default)
-		)
-	)
-	(wire
-		(pts
 			(xy 81.28 105.41) (xy 99.06 105.41)
 		)
@@
 	(wire
 		(pts
-			(xy 218.44 41.91) (xy 226.06 41.91)
+			(xy 218.44 41.91) (xy 252.73 41.91)
 		)
 		(stroke
@@
 				(path "/5cbb45d4-7f83-48dd-a53b-5c75c7d1d827/acc6b550-0215-4302-88ee-d8cdb26529cb"
 					(reference "#PWR056")
-					(unit 1)
-				)
-			)
-		)
-	)
-	(symbol
-		(lib_id "Device:NetTie_2")
-		(at 229.87 60.96 0)
-		(unit 1)
-		(exclude_from_sim no)
-		(in_bom no)
-		(on_board yes)
-		(dnp no)
-		(fields_autoplaced yes)
-		(property "Reference" "NT6"
-			(at 229.87 55.88 0)
-			(effects
-				(font
-					(size 1.27 1.27)
-				)
-			)
-		)
-		(property "Value" "NetTie_2"
-			(at 229.87 58.42 0)
-			(effects
-				(font
-					(size 1.27 1.27)
-				)
-			)
-		)
-		(property "Footprint" ""
-			(at 229.87 60.96 0)
-			(effects
-				(font
-					(size 1.27 1.27)
-				)
-				(hide yes)
-			)
-		)
-		(property "Datasheet" "~"
-			(at 229.87 60.96 0)
-			(effects
-				(font
-					(size 1.27 1.27)
-				)
-				(hide yes)
-			)
-		)
-		(property "Description" "Net tie, 2 pins"
-			(at 229.87 60.96 0)
-			(effects
-				(font
-					(size 1.27 1.27)
-				)
-				(hide yes)
-			)
-		)
-		(pin "1"
-		)
-		(pin "2"
-		)
-		(instances
-			(project ""
-				(path "/5cbb45d4-7f83-48dd-a53b-5c75c7d1d827/acc6b550-0215-4302-88ee-d8cdb26529cb"
-					(reference "NT6")
 					(unit 1)
 				)
@@
 					(unit 1)
 				)
-			)
-		)
-	)
-	(symbol
-		(lib_id "Device:NetTie_2")
-		(at 228.6 41.91 0)
-		(unit 1)
-		(exclude_from_sim no)
-		(in_bom no)
-		(on_board yes)
-		(dnp no)
-		(fields_autoplaced yes)
-		(property "Reference" "NT5"
-			(at 228.6 36.83 0)
-			(effects
-				(font
-					(size 1.27 1.27)
-				)
-			)
-		)
-		(property "Value" "NetTie_2"
-			(at 228.6 39.37 0)
-			(effects
-				(font
-					(size 1.27 1.27)
-				)
-			)
-		)
-		(property "Footprint" ""
-			(at 228.6 41.91 0)
-			(effects
-				(font
-					(size 1.27 1.27)
-				)
-				(hide yes)
-			)
-		)
-		(property "Datasheet" "~"
-			(at 228.6 41.91 0)
-			(effects
-				(font
-					(size 1.27 1.27)
-				)
-				(hide yes)
-			)
-		)
-		(property "Description" "Net tie, 2 pins"
-			(at 228.6 41.91 0)
-			(effects
-				(font
-					(size 1.27 1.27)
-				)
-				(hide yes)
-			)
-		)
-		(pin "1"
-		)
-		(pin "2"
-		)
-		(instances
-			(project ""
-				(path "/5cbb45d4-7f83-48dd-a53b-5c75c7d1d827/acc6b550-0215-4302-88ee-d8cdb26529cb"
-					(reference "NT5")
-					(unit 1)
-				)
