File: v0.3/sound_pwm.kicad_sch (KiCad schematic)
At the start: 1 part, among them J6 SPEAKER_CONNECTOR

Commit message: v0.3: lots of routing done
Parts:
- J6: footprint Connector_PinHeader_2.54mm:PinHeader_1x02_P2.54mm_Vertical -> Resistor_SMD:R_0603_1608Metric
Changed lines of the file:
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@@
 			)
 		)
-		(property "Footprint" "Connector_PinHeader_2.54mm:PinHeader_1x02_P2.54mm_Vertical"
+		(property "Footprint" "Resistor_SMD:R_0603_1608Metric"
 			(at 118.11 76.2 0)
 			(effects
