File: v0.3/power_smps.kicad_sch (KiCad schematic)
At the start: 24 parts, among them IC3 BQ25628ERYKR, IC4 RT6150B-33GQW

Commit message: v0.3: lots of routing done
Parts:
- TH1: footprint Resistor_SMD:R_0402_1005Metric -> CustomFootprints:R_0402_1005Metric_Sunken
Changed lines of the file:
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@@
 			)
 		)
-		(property "Footprint" "Resistor_SMD:R_0402_1005Metric"
+		(property "Footprint" "CustomFootprints:R_0402_1005Metric_Sunken"
 			(at 59.69 111.76 0)
 			(effects

Commit message: v0.3: DRC checks mostly pass, onto final tweaks
Parts:
- TP1: footprint TestPoint:TestPoint_Pad_2.5x2.5mm -> TestPoint:TestPoint_Pad_1.0x1.0mm
Changed lines of the file:
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@@
 			)
 		)
-		(property "Footprint" "TestPoint:TestPoint_Pad_2.5x2.5mm"
+		(property "Footprint" "TestPoint:TestPoint_Pad_1.0x1.0mm"
 			(at 48.26 58.42 0)
 			(effects
