File: rp2350-v0.2/rp2350-v0.2.kicad_pcb (KiCad board)
At the start: 4 copper layers, 65 x 65 mm, 118 parts, among them IC1 M95512-RMN6TP, IC2 TFBS4711-TT1, IC3 BQ25628ERYKR, IC4 RT6150B-33GQW, IC5 W25Q128JVSIM_TR, J1 USB4215-03-A, J2 SWD, J3 BAT, J4 DO0180FMST08, J5 UART, J6 SPEAKER_CONNECTOR, SW1 BUT_R, SW2 BUT_M, SW3 BUT_L, SW4 RUN, SW5 BOOTSEL, U1 RP2350A-QFN60, Y1 ABM8-272-T3, Y2 SIT1533AI-H4-DCC-32.768E

Commit message: v0.2: move files around
Parts:
- moved C34 7.89 mm to (139.9, 82.0)
- moved C35 7.86 mm to (139.9, 81.0)
- moved C22 7.85 mm to (133.8, 77.1)
- moved C27 7.85 mm to (133.8, 76.1)
- moved TP2 2.20 mm to (140.0, 86.2)
Routing:
- net /buttons/BUT_R_1: track 3.23 -> 11.2 mm
- net GND: track 25.2 -> 31.4 mm, vias 213 -> 214
- net /mcu/MCU_1V1: track 31.6 -> 36.7 mm
- net /mcu/MCU_3V3: track 38.7 -> 42.2 mm
- net /mcu/VREG_LX: track 0.00 -> 0.55 mm
Other:
- board text added: "picowalker v0.2.1"
- board text added: "picowalker v0.2.1 by mamba2410"
- board text removed: "picowalker v0.2"
- board text removed: "picowalker v0.2 by mamba2410"
