File: picowalker-v0.4/accel_bma400.kicad_sch (KiCad schematic)
At the start: 0 parts

Commit message: v0.4: schematic laid out first draft
Parts:
- added C20, C21: 4.7u, Capacitor_SMD:C_0402_1005Metric, symbol Device:C
- added U3: BMA400, symbol picowalker:BMA400
Connections:
- new net +3.3V: C20.1, C21.1, U3.3 (VDDIO), U3.7 (VDD)
- new net GND: C20.2, C21.2, U3.8 (GNDIO), U3.9 (GND)
- new net INT: U3.5 (INT1)
- new net MISO: U3.1 (SDO)
- new net MOSI: U3.2 (SDX)
- new net SCK: U3.12 (SCX)
- new net ~{CS}: U3.10 (~{CS})
- no-connect marks 0 -> 1

Commit message: v0.4: first rough placement of PCB
Parts:
- U3: footprint (none) -> picowalker:BOSCH_LGA-12_BMA400
Changed lines of the file:
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@@
 			)
 		)
-		(property "Footprint" ""
+		(property "Footprint" "picowalker:BOSCH_LGA-12_BMA400"
 			(at 115.57 63.5 0)
 			(effects

Commit message: v0.4: good start on routing
Connections:
- net MISO renamed SPI.MISO
- net MOSI renamed SPI.MOSI
- net SCK renamed SPI.SCK
Changed lines of the file:
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@@
 		)
 	)
-	(label "MOSI"
+	(label "SPI.MOSI"
 		(at 95.25 74.93 0)
 		(effects
@@
 		)
 	)
-	(label "SCK"
+	(label "SPI.SCK"
 		(at 95.25 80.01 0)
 		(effects
@@
 		)
 	)
-	(label "MISO"
+	(label "SPI.MISO"
 		(at 95.25 77.47 0)
 		(effects

Commit message: v0.4: drc mostly done, need to fiddle with TH1
Parts:
- C20, C21: value 4.7u -> 0.1u
Changed lines of the file:
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@@
 			)
 		)
-		(property "Value" "4.7u"
+		(property "Value" "0.1u"
 			(at 57.15 44.4499 0)
 			(effects
@@
 			)
 		)
-		(property "Value" "4.7u"
+		(property "Value" "0.1u"
 			(at 39.37 44.4499 0)
 			(effects
