File: picowalker-v0.4/connectors.kicad_sch (KiCad schematic)
At the start: 0 parts

Commit message: v0.4: schematic laid out first draft
Parts:
- added J1: 12402012E212A, symbol Connector:USB_C_Receptacle_USB2.0_16P
- added J2: BAT, Connector_Molex:Molex_PicoBlade_53261-0271_1x02-1MP_P1.25mm_Horizontal, symbol Connector_Generic:Conn_01x02
- added J3: SWD, Connector_JST:JST_SH_SM03B-SRSS-TB_1x03-1MP_P1.00mm_Horizontal, symbol Connector_Generic:Conn_01x03
- added J4: UART, Connector_JST:JST_SH_SM03B-SRSS-TB_1x03-1MP_P1.00mm_Horizontal, symbol Connector_Generic:Conn_01x03
- added R7, R8: 5.1k, Resistor_SMD:R_0402_1005Metric, symbol Device:R
Connections:
- new net BAT+: J2.1 (Pin_1)
- new net CC1: J1.A5 (CC1), R7.1
- new net CC2: J1.B5 (CC2), R8.1
- new net DN: J1.A7 (D-), J1.B7 (D-)
- new net DP: J1.A6 (D+), J1.B6 (D+)
- new net GND: J1.A1 (GND), J1.A12 (GND), J1.B1 (GND), J1.B12 (GND), J1.S1 (SHIELD), J2.2 (Pin_2), J3.2 (Pin_2), J4.2 (Pin_2), R7.2, R8.2
- new net RX: J4.1 (Pin_1)
- new net SWCLK: J3.1 (Pin_1)
- new net SWDIO: J3.3 (Pin_3)
- new net TX: J4.3 (Pin_3)
- new net VBUS: J1.A4 (VBUS), J1.A9 (VBUS), J1.B4 (VBUS), J1.B9 (VBUS)
- no-connect marks 0 -> 2
Other:
- note added: "Amphenol 12402012E212A"
- note added: "Mates with: - 151340200 cable assembly - 510210200 connector"
- note added: "Molex 53261-0271"

Commit message: v0.4: first rough placement of PCB
Parts:
- J1: footprint (none) -> picowalker:USBC
Connections:
- net DN renamed USB.DN
- net DP renamed USB.DP
Changed lines of the file:
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@@
 		)
 	)
-	(label "DP"
+	(label "USB.DP"
 		(at 74.93 57.15 0)
 		(effects
@@
 		)
 	)
-	(label "DN"
+	(label "USB.DN"
 		(at 74.93 52.07 0)
 		(effects
@@
 			)
 		)
-		(property "Footprint" ""
+		(property "Footprint" "picowalker:USBC"
 			(at 54.61 52.07 0)
 			(effects

Commit message: v0.4: good start on routing
Parts:
- added U8: DT1240-04LP-7, picowalker:U-DFN2510-10, symbol picowalker:DT1240-04LP-7
Connections:
- net GND: now also U8.3 (VSS), U8.8 (VSS)
- net USB.DN: now also U8.1 (IO1)
- net USB.DP: now also U8.2 (IO2)
- net VBUS: now also U8.5 (IO4)
- net RX renamed DBG_UART.RX
- net SWCLK renamed SWD.SWCLK
- net SWDIO renamed SWD.SWDIO
- net TX renamed DBG_UART.TX
- no-connect marks 2 -> 3

Commit message: v0.4: running DRC checks
Parts:
- U8: footprint picowalker:U-DFN2510-10 -> picowalker:U-DFN2510-10_oneside
Connections:
- net VBUS: now also U8.4 (IO3); no longer U8.5 (IO4)

Commit message: v0.4: drc mostly done, need to fiddle with TH1
Parts:
- J3, J4: footprint Connector_JST:JST_SH_SM03B-SRSS-TB_1x03-1MP_P1.00mm_Horizontal -> picowalker:JST_SH_SM03B-SRSS-TB_1x03-1MP_P1.00mm_Horizontal_wider
Other:
- note added: "ESD protection"
Changed lines of the file:
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@@
 	(generator_version "9.0")
 	(paper "A4")
+	(text "ESD protection"
+		(exclude_from_sim no)
+		(at 108.204 58.42 0)
+		(effects
+			(font
+				(size 1.27 1.27)
+			)
+		)
+	)
 	(text "Mates with:\n- 151340200 cable assembly\n- 510210200 connector"
 		(exclude_from_sim no)
@@
 			)
 		)
-		(property "Footprint" "Connector_JST:JST_SH_SM03B-SRSS-TB_1x03-1MP_P1.00mm_Horizontal"
+		(property "Footprint" "picowalker:JST_SH_SM03B-SRSS-TB_1x03-1MP_P1.00mm_Horizontal_wider"
 			(at 204.47 128.27 0)
 			(effects
@@
 			)
 		)
-		(property "Footprint" "Connector_JST:JST_SH_SM03B-SRSS-TB_1x03-1MP_P1.00mm_Horizontal"
+		(property "Footprint" "picowalker:JST_SH_SM03B-SRSS-TB_1x03-1MP_P1.00mm_Horizontal_wider"
 			(at 167.64 58.42 0)
 			(effects

Commit message: v0.4: update readme and add renders
Parts:
- J1: footprint picowalker:USBC -> Connector_USB:USB_C_Receptacle_GCT_USB4105-xx-A_16P_TopMnt_Horizontal
Changed lines of the file:
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@@
 			)
 		)
-		(property "Footprint" "picowalker:USBC"
+		(property "Footprint" "Connector_USB:USB_C_Receptacle_GCT_USB4105-xx-A_16P_TopMnt_Horizontal"
 			(at 54.61 52.07 0)
 			(effects
