File: picowalker-v0.4/eeprom_m95512.kicad_sch (KiCad schematic)
At the start: 0 parts

Commit message: v0.4: schematic laid out first draft
Parts:
- added C22: 4.7u, Capacitor_SMD:C_0402_1005Metric, symbol Device:C
- added R15, R16: 5.1k, Resistor_SMD:R_0402_1005Metric, symbol Device:R
- added U4: M95512DxMC, symbol picowalker:M95512DxMC
Connections:
- new net +3.3V: C22.1, R15.1, U4.3 (~{W}/~{WP}), U4.7 (~{HOLD}), U4.8 (VCC)
- new net GND: C22.2, R16.2, U4.4 (GND), U4.9 (EPAD)
- new net MISO: U4.2 (Q/MISO)
- new net MOSI: U4.5 (D/MOSI)
- new net SCK: R16.1, U4.6 (C/SCK)
- new net ~{CS}: R15.2, U4.1 (~{S}/~{CS})

Commit message: v0.4: first rough placement of PCB
Parts:
- U4: footprint (none) -> picowalker:XDFN8
Changed lines of the file:
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@@
 			)
 		)
-		(property "Footprint" ""
+		(property "Footprint" "picowalker:XDFN8"
 			(at 124.46 80.01 0)
 			(effects

Commit message: v0.4: good start on routing
Parts:
- U4: footprint picowalker:XDFN8 -> picowalker:UFDFPN8
Connections:
- net MISO renamed SPI.MISO
- net MOSI renamed SPI.MOSI
- net SCK renamed SPI.SCK
Other:
- note added: "Consider M95M01-DWMN or CAV25M01 for 128kB Both are pin-compatible with M95512-DWMN in SO8 4.9 x 6.0 mm package"
Changed lines of the file:
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@@
 	(generator_version "9.0")
 	(paper "A4")
+	(text "Consider M95M01-DWMN or CAV25M01 for 128kB\nBoth are pin-compatible with M95512-DWMN in SO8 4.9 x 6.0 mm package"
+		(exclude_from_sim no)
+		(at 127 64.008 0)
+		(effects
+			(font
+				(size 1.27 1.27)
+			)
+		)
+	)
 	(text_box "Decoupling and bulk"
 		(exclude_from_sim no)
@@
 		)
 	)
-	(label "MOSI"
+	(label "SPI.MOSI"
 		(at 139.7 88.9 0)
 		(effects
@@
 		)
 	)
-	(label "SCK"
+	(label "SPI.SCK"
 		(at 139.7 93.98 0)
 		(effects
@@
 		)
 	)
-	(label "MISO"
+	(label "SPI.MISO"
 		(at 139.7 91.44 0)
 		(effects
@@
 			)
 		)
-		(property "Footprint" "picowalker:XDFN8"
+		(property "Footprint" "picowalker:UFDFPN8"
 			(at 124.46 80.01 0)
 			(effects

Commit message: v0.4: drc mostly done, need to fiddle with TH1
Parts:
- R16: now left out of the parts list
Other:
- note added: "Hardware pullup required. If ~{CS} isn't driven at any time, chip will malfunction and will not be recoverable until power cycle. See ST's AN2014 section 4.2"
- note added: "MN = SO8N MC = UFDFPN8"
- note added: "Pulldown only required if host releases ~{CS} while SCK is still clocking."
Changed lines of the file:
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@@
 	(generator_version "9.0")
 	(paper "A4")
+	(text "MN = SO8N\nMC = UFDFPN8"
+		(exclude_from_sim no)
+		(at 135.89 72.39 0)
+		(effects
+			(font
+				(size 1.27 1.27)
+			)
+			(justify left top)
+		)
+	)
 	(text "Consider M95M01-DWMN or CAV25M01 for 128kB\nBoth are pin-compatible with M95512-DWMN in SO8 4.9 x 6.0 mm package"
 		(exclude_from_sim no)
-		(at 127 64.008 0)
-		(effects
-			(font
-				(size 1.27 1.27)
-			)
+		(at 127.254 48.26 0)
+		(effects
+			(font
+				(size 1.27 1.27)
+			)
+		)
+	)
+	(text "Pulldown only required if host releases ~{CS} while SCK is still clocking."
+		(exclude_from_sim no)
+		(at 147.066 100.076 0)
+		(effects
+			(font
+				(size 1.27 1.27)
+			)
+			(justify left top)
+		)
+	)
+	(text "Hardware pullup required.\nIf ~{CS} isn't driven at any time, chip will malfunction\nand will not be recoverable until power cycle.\nSee ST's AN2014 section 4.2"
+		(exclude_from_sim no)
+		(at 43.688 78.74 0)
+		(effects
+			(font
+				(size 1.27 1.27)
+			)
+			(justify left top)
 		)
 	)
@@
 		(unit 1)
 		(exclude_from_sim no)
-		(in_bom yes)
+		(in_bom no)
 		(on_board yes)
 		(dnp yes)
