File: picowalker-v0.4/flash_w25q128.kicad_sch (KiCad schematic)
At the start: 0 parts

Commit message: v0.4: schematic laid out first draft
Parts:
- added C15: 0.1u, Capacitor_SMD:C_0402_1005Metric, symbol Device:C
- added C16: 4.7u, Capacitor_SMD:C_0402_1005Metric, symbol Device:C
- added U2: W25Q128JVP, Package_SON:WSON-8-1EP_6x5mm_P1.27mm_EP3.4x4.3mm, symbol Memory_Flash:W25Q128JVP
Connections:
- new net +3.3V: C15.1, C16.1, U2.8 (VCC)
- new net GND: C15.2, C16.2, U2.4 (GND), U2.9 (EP)
- new net SCK: U2.6 (CLK)
- new net SD0: U2.5 (DI/IO_{0})
- new net SD1: U2.2 (DO/IO_{1})
- new net SD2: U2.3 (~{WP}/IO_{2})
- new net SD3: U2.7 (~{HOLD}/~{RESET}/IO_{3})
- new net ~{CS}: U2.1 (~{CS})

Commit message: v0.4: more rationalisation
Parts:
- C15: now not fitted
Changed lines of the file:
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@@
 		(in_bom yes)
 		(on_board yes)
-		(dnp no)
+		(dnp yes)
 		(property "Reference" "C15"
 			(at 46.99 48.2599 0)

Commit message: v0.4: good start on routing
Parts:
- removed C15: 0.1u, Capacitor_SMD:C_0402_1005Metric, symbol Device:C
Connections:
- net SCK renamed QSPI.SCK
- net SD0 renamed QSPI.SD0
- net SD1 renamed QSPI.SD1
- net SD2 renamed QSPI.SD2
- net SD3 renamed QSPI.SD3
Other:
- moved on the sheet: C16
Changed lines of the file:
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@@
-		(color 0 0 0 0)
-	)
-	(junction
-		(at 55.88 54.61)
-		(diameter 0)
-		(color 0 0 0 0)
-	)
-	(junction
-		(at 55.88 44.45)
-		(diameter 0)
 		(color 0 0 0 0)
 	)
@@
 	(wire
 		(pts
-			(xy 60.96 45.72) (xy 60.96 44.45)
+			(xy 55.88 43.18) (xy 55.88 45.72)
 		)
 		(stroke
@@
 		)
 	)
-	(wire
-		(pts
-			(xy 50.8 45.72) (xy 50.8 44.45)
-		)
-		(stroke
-			(width 0)
-			(type default)
-		)
-	)
 	(bus
 		(pts
@@
 	(wire
 		(pts
-			(xy 60.96 54.61) (xy 55.88 54.61)
-		)
-		(stroke
-			(width 0)
-			(type default)
-		)
-	)
-	(wire
-		(pts
 			(xy 101.6 88.9) (xy 118.11 88.9)
 		)
@@
 	(wire
 		(pts
-			(xy 55.88 44.45) (xy 55.88 43.18)
-		)
-		(stroke
-			(width 0)
-			(type default)
-		)
-	)
-	(wire
-		(pts
-			(xy 50.8 53.34) (xy 50.8 54.61)
-		)
-		(stroke
-			(width 0)
-			(type default)
-		)
-	)
-	(wire
-		(pts
-			(xy 50.8 54.61) (xy 55.88 54.61)
-		)
-		(stroke
-			(width 0)
-			(type default)
-		)
-	)
-	(wire
-		(pts
 			(xy 104.14 96.52) (xy 118.11 96.52)
 		)
@@
 	(wire
 		(pts
-			(xy 60.96 44.45) (xy 55.88 44.45)
-		)
-		(stroke
-			(width 0)
-			(type default)
-		)
-	)
-	(wire
-		(pts
 			(xy 128.27 77.47) (xy 128.27 83.82)
 		)
@@
 	(wire
 		(pts
-			(xy 60.96 53.34) (xy 60.96 54.61)
-		)
-		(stroke
-			(width 0)
-			(type default)
-		)
-	)
-	(wire
-		(pts
-			(xy 50.8 44.45) (xy 55.88 44.45)
-		)
-		(stroke
-			(width 0)
-			(type default)
-		)
-	)
-	(wire
-		(pts
-			(xy 55.88 54.61) (xy 55.88 55.88)
+			(xy 55.88 53.34) (xy 55.88 55.88)
 		)
 		(stroke
@@
 		)
 	)
-	(label "SD3"
-		(at 110.49 101.6 0)
+	(label "QSPI.SD3"
+		(at 106.68 101.6 0)
 		(effects
 			(font
@@
 		)
 	)
-	(label "SD0"
-		(at 110.49 93.98 0)
+	(label "QSPI.SD0"
+		(at 106.68 93.98 0)
 		(effects
 			(font
@@
 		)
 	)
-	(label "SCK"
-		(at 110.49 91.44 0)
+	(label "QSPI.SCK"
+		(at 106.68 91.44 0)
 		(effects
 			(font
@@
 		)
 	)
-	(label "SD2"
-		(at 110.49 99.06 0)
+	(label "QSPI.SD2"
+		(at 106.68 99.06 0)
 		(effects
 			(font
@@
 		)
 	)
-	(label "SD1"
-		(at 110.49 96.52 0)
+	(label "QSPI.SD1"
+		(at 106.68 96.52 0)
 		(effects
 			(font
@@
 	(symbol
 		(lib_id "Device:C")
-		(at 60.96 49.53 0)
+		(at 55.88 49.53 0)
 		(unit 1)
 		(exclude_from_sim no)
@@
 		(fields_autoplaced yes)
 		(property "Reference" "C16"
-			(at 64.77 48.2599 0)
+			(at 59.69 48.2599 0)
 			(effects
 				(font
@@
 		)
 		(property "Value" "4.7u"
-			(at 64.77 50.7999 0)
+			(at 59.69 50.7999 0)
 			(effects
 				(font
@@
 		)
 		(property "Footprint" "Capacitor_SMD:C_0402_1005Metric"
-			(at 61.9252 53.34 0)
+			(at 56.8452 53.34 0)
 			(effects
 				(font
@@
 		)
 		(property "Datasheet" "~"
-			(at 60.96 49.53 0)
+			(at 55.88 49.53 0)
 			(effects
 				(font
@@
 		)
 		(property "Description" "Unpolarized capacitor"
-			(at 60.96 49.53 0)
+			(at 55.88 49.53 0)
 			(effects
 				(font
@@
 					(unit 1)
 				)
-			)
-		)
-	)
-	(symbol
-		(lib_id "Device:C")
-		(at 50.8 49.53 0)
-		(unit 1)
-		(exclude_from_sim no)
-		(in_bom yes)
-		(on_board yes)
-		(dnp yes)
-		(property "Reference" "C15"
-			(at 46.99 48.2599 0)
-			(effects
-				(font
-					(size 1.27 1.27)
-				)
-				(justify right)
-			)
-		)
-		(property "Value" "0.1u"
-			(at 46.99 50.7999 0)
-			(effects
-				(font
-					(size 1.27 1.27)
-				)
-				(justify right)
-			)
-		)
-		(property "Footprint" "Capacitor_SMD:C_0402_1005Metric"
-			(at 51.7652 53.34 0)
-			(effects
-				(font
-					(size 1.27 1.27)
-				)
-				(hide yes)
-			)
-		)
-		(property "Datasheet" "~"
-			(at 50.8 49.53 0)
-			(effects
-				(font
-					(size 1.27 1.27)
-				)
-				(hide yes)
-			)
-		)
-		(property "Description" "Unpolarized capacitor"
-			(at 50.8 49.53 0)
-			(effects
-				(font
-					(size 1.27 1.27)
-				)
-				(hide yes)
-			)
-		)
-		(pin "2"
-		)
-		(pin "1"
-		)
-		(instances
-			(project ""
-				(path "/aa8773bf-a88b-4bf9-9961-8e312cd9d0e3/7a794e87-c7b9-4c3e-ac66-3fc5c41c1724"
-					(reference "C15")
-					(unit 1)
-				)
