File: picowalker-v0.4/irda_tfdu4711_pio.kicad_sch (KiCad schematic)
At the start: 0 parts

Commit message: v0.4: schematic laid out first draft
Parts:
- added C23: 0.1u, Capacitor_SMD:C_0402_1005Metric, symbol Device:C
- added C24: 4.7u, Capacitor_SMD:C_0402_1005Metric, symbol Device:C
- added R17: 56R, Resistor_SMD:R_0402_1005Metric, symbol Device:R
- added R18: 47R, Resistor_SMD:R_0402_1005Metric, symbol Device:R
- added U5: TFBS4711, symbol picowalker:TFBS4711
Connections:
- new net +3.3V: C24.1, R17.1, R18.1
- new net GND: C23.2, C24.2, U5.6 (GND)
- new net RX: U5.3 (RXD)
- new net SD: U5.4 (SD)
- new net TX: U5.2 (TXD)
- new net VCC1: C23.1, R18.2, U5.5 (VCC1)
- new net VCC2: R17.2, U5.1 (VCC2)
Other:
- note added: "Expect serial to be encoded with IrDA. MCU can do this with PIO or IrDA mode in UART"

Commit message: v0.4: more rationalisation
Parts:
- R17: value 56R -> 47R
Changed lines of the file:
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@@
 			)
 		)
-		(property "Value" "56R"
+		(property "Value" "47R"
 			(at 58.42 35.56 90)
 			(effects

Commit message: v0.4: first rough placement of PCB
Parts:
- U5: footprint (none) -> picowalker:TFBS4711-TR
Changed lines of the file:
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@@
 			)
 		)
-		(property "Footprint" ""
+		(property "Footprint" "picowalker:TFBS4711-TR"
 			(at 160.02 46.99 0)
 			(effects

Commit message: v0.4: good start on routing
Connections:
- net RX renamed IRDA.RX
- net TX renamed IRDA.TX
Other:
- note added: "Bulk capacitance and current limit"
- note added: "Low pass filter"
Changed lines of the file:
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@@
+		)
+	)
+	(text "Bulk capacitance and current limit"
+		(exclude_from_sim no)
+		(at 61.468 29.21 0)
+		(effects
+			(font
+				(size 1.27 1.27)
+			)
+		)
+	)
+	(text "Low pass filter"
+		(exclude_from_sim no)
+		(at 57.658 65.024 0)
+		(effects
+			(font
+				(size 1.27 1.27)
+			)
 		)
 	)
@@
 		)
 	)
-	(label "RX"
-		(at 143.51 62.23 0)
+	(label "IRDA.RX"
+		(at 140.97 62.23 0)
 		(effects
 			(font
@@
 		)
 	)
-	(label "TX"
-		(at 143.51 59.69 0)
-		(effects
-			(font
+	(label "IRDA.TX"
+		(at 140.97 59.69 0)
+		(effects
+			(font

Commit message: v0.4: drc mostly done, need to fiddle with TH1
Other:
- note added: "From app note under "emitter signal timing" "since the receiver saturates during transmission, it is also necessary to include a latency time of > 150 μs after transmission before the receiver is ready for reception again""
- note added: "Original uses IrDA SIR V1.0 at 115200 baud, so we do the same."
- note added: "See Vishay's app note on reference layouts https://www.vishay.com/docs/82610/referencelayoutscircuitdiagrams.pdf R17 is a current limiting resistor. 47R resistor gives IRED forward current of around 40-50 mA at 3.3 V. This is 132-150 mW, more than the common 1/16 W (62.5 mW) power rating for resistors. From testing, this seems to be fine since its pulsed. Intensity is at around 15%. 100R resistor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"
- moved on the sheet: U5
Changed lines of the file:
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@@
 	(generator_version "9.0")
 	(paper "A4")
+	(text "Original uses IrDA SIR V1.0 at 115200 baud, so we do the same."
+		(exclude_from_sim no)
+		(at 22.352 98.552 0)
+		(effects
+			(font
+				(size 1.27 1.27)
+			)
+			(justify left)
+		)
+	)
 	(text "Expect serial to be encoded with IrDA.\nMCU can do this with PIO or IrDA mode in UART"
 		(exclude_from_sim no)
-		(at 97.536 50.292 0)
+		(at 115.57 66.04 0)
 		(effects
 			(font
@@
 				(size 1.27 1.27)
 			)
+		)
+	)
+	(text "See Vishay's app note on reference layouts\nhttps://www.vishay.com/docs/82610/referencelayoutscircuitdiagrams.pdf\n\nR17 is a current limiting resistor.\n\n47R resistor gives IRED forward current of around 40-50 mA at 3.3 V.\nThis is 132-150 mW, more than the common 1/16 W (62.5 mW) power rating for resistors.\nFrom testing, this seems to be fine since its pulsed.\nIntensity is at around 15%.\n\n100R resistor is 20 mA, or 66 mW, and <10% intensity.\n\nDatasheet says to expect <2 mA average current whtn I_{IRED} (IRED forward current)\nis 300 mA and a 20% duty cycle.\n"
+		(exclude_from_sim no)
+		(at 92.456 22.606 0)
+		(effects
+			(font
+				(size 1.27 1.27)
+			)
+			(justify left top)
+		)
+	)
+	(text "From app note under \"emitter signal timing\"\n\n\"since the receiver saturates during transmission, it is also necessary to include a latency time of > 150 μs after transmission\nbefore the receiver is ready for reception again\""
+		(exclude_from_sim no)
+		(at 22.606 110.998 0)
+		(effects
+			(font
+				(size 1.27 1.27)
+			)
+			(justify left)
 		)
 	)
@@
 	)
 	(bus_entry
-		(at 137.16 59.69)
+		(at 153.67 76.2)
 		(size 2.54 2.54)
 		(stroke
@@
 	)
 	(bus_entry
-		(at 137.16 57.15)
+		(at 153.67 73.66)
 		(size 2.54 2.54)
 		(stroke
@@
 	(wire
 		(pts
-			(xy 139.7 62.23) (xy 149.86 62.23)
+			(xy 156.21 78.74) (xy 166.37 78.74)
 		)
 		(stroke
@@
 	(bus
 		(pts
-			(xy 137.16 57.15) (xy 137.16 59.69)
+			(xy 153.67 73.66) (xy 153.67 76.2)
 		)
 		(stroke
@@
 	(bus
 		(pts
-			(xy 137.16 54.61) (xy 137.16 57.15)
-		)
-		(stroke
-			(width 0)
-			(type default)
-		)
-	)
-	(wire
-		(pts
-			(xy 139.7 64.77) (xy 149.86 64.77)
-		)
-		(stroke
-			(width 0)
-			(type default)
-		)
-	)
-	(wire
-		(pts
-			(xy 151.13 45.72) (xy 157.48 45.72)
-		)
-		(stroke
-			(width 0)
-			(type default)
-		)
-	)
-	(wire
-		(pts
-			(xy 139.7 59.69) (xy 149.86 59.69)
-		)
-		(stroke
-			(width 0)
-			(type default)
-		)
-	)
-	(wire
-		(pts
-			(xy 156.21 40.64) (xy 162.56 40.64)
-		)
-		(stroke
-			(width 0)
-			(type default)
-		)
-	)
-	(wire
-		(pts
-			(xy 162.56 40.64) (xy 162.56 48.26)
+			(xy 153.67 71.12) (xy 153.67 73.66)
+		)
+		(stroke
+			(width 0)
+			(type default)
+		)
+	)
+	(wire
+		(pts
+			(xy 156.21 81.28) (xy 166.37 81.28)
+		)
+		(stroke
+			(width 0)
+			(type default)
+		)
+	)
+	(wire
+		(pts
+			(xy 167.64 62.23) (xy 173.99 62.23)
+		)
+		(stroke
+			(width 0)
+			(type default)
+		)
+	)
+	(wire
+		(pts
+			(xy 156.21 76.2) (xy 166.37 76.2)
+		)
+		(stroke
+			(width 0)
+			(type default)
+		)
+	)
+	(wire
+		(pts
+			(xy 172.72 57.15) (xy 179.07 57.15)
+		)
+		(stroke
+			(width 0)
+			(type default)
+		)
+	)
+	(wire
+		(pts
+			(xy 179.07 57.15) (xy 179.07 64.77)
 		)
 		(stroke
@@
 	(wire
 		(pts
-			(xy 160.02 74.93) (xy 160.02 80.01)
+			(xy 176.53 91.44) (xy 176.53 96.52)
 		)
 		(stroke
@@
 	(wire
 		(pts
-			(xy 157.48 45.72) (xy 157.48 48.26)
+			(xy 173.99 62.23) (xy 173.99 64.77)
 		)
 		(stroke
@@
 	)
 	(label "IRDA.RX"
-		(at 140.97 62.23 0)
+		(at 157.48 78.74 0)
 		(effects
 			(font
@@
 	)
 	(label "VCC1"
-		(at 156.21 40.64 0)
+		(at 172.72 57.15 0)
 		(effects
 			(font
@@
 	)
 	(label "IRDA.TX"
-		(at 140.97 59.69 0)
+		(at 157.48 76.2 0)
 		(effects
 			(font
@@
 	)
 	(label "VCC2"
-		(at 151.13 45.72 0)
+		(at 167.64 62.23 0)
 		(effects
 			(font
@@
 	(hierarchical_label "SD"
 		(shape input)
-		(at 139.7 64.77 180)
+		(at 156.21 81.28 180)
 		(effects
 			(font
@@
 	(hierarchical_label "IRDA{SERIAL}"
 		(shape bidirectional)
-		(at 137.16 54.61 180)
+		(at 153.67 71.12 180)
 		(effects
 			(font
@@
 	(symbol
 		(lib_id "picowalker:TFBS4711")
-		(at 160.02 46.99 0)
+		(at 176.53 63.5 0)
 		(unit 1)
 		(exclude_from_sim no)
@@
 		(fields_autoplaced yes)
 		(property "Reference" "U5"
-			(at 168.91 60.3249 0)
+			(at 185.42 76.8349 0)
 			(effects
 				(font
@@
 		)
 		(property "Value" "TFBS4711"
-			(at 168.91 62.8649 0)
+			(at 185.42 79.3749 0)
 			(effects
 				(font
@@
 		)
 		(property "Footprint" "picowalker:TFBS4711-TR"
-			(at 160.02 46.99 0)
+			(at 176.53 63.5 0)
 			(effects
 				(font
@@
 		)
 		(property "Datasheet" ""
-			(at 160.02 46.99 0)
+			(at 176.53 63.5 0)
 			(effects
 				(font
@@
 		)
 		(property "Description" ""
-			(at 160.02 46.99 0)
+			(at 176.53 63.5 0)
 			(effects
 				(font
@@
 	(symbol
 		(lib_id "power:GND")
-		(at 160.02 80.01 0)
+		(at 176.53 96.52 0)
 		(unit 1)
 		(exclude_from_sim no)
@@
 		(fields_autoplaced yes)
 		(property "Reference" "#PWR053"
-			(at 160.02 86.36 0)
+			(at 176.53 102.87 0)
 			(effects
 				(font
@@
 		)
 		(property "Value" "GND"
-			(at 160.02 85.09 0)
+			(at 176.53 101.6 0)
 			(effects
 				(font
@@
 		)
 		(property "Footprint" ""
-			(at 160.02 80.01 0)
+			(at 176.53 96.52 0)
 			(effects
 				(font
@@
 		)
 		(property "Datasheet" ""
-			(at 160.02 80.01 0)
+			(at 176.53 96.52 0)
 			(effects
 				(font
@@
 		)
 		(property "Description" "Power symbol creates a global label with name \"GND\" , ground"
-			(at 160.02 80.01 0)
-			(effects
-				(font
+			(at 176.53 96.52 0)
+			(effects
+				(font
