File: picowalker-v0.4/rtc_sit1533.kicad_sch (KiCad schematic)
At the start: 0 parts

Commit message: v0.4: schematic laid out first draft
Parts:
- added Y2: SIT1533AI-H4-DCC-32.768E, symbol picowalker:SIT1533AI-H4-DCC-32.768E
Connections:
- new net +3.3V: Y2.4 (VDD)
- new net CLK: Y2.3 (CLK_OUT)
- new net GND: Y2.2 (GND)

Commit message: v0.4: first rough placement of PCB
Parts:
- Y2: footprint (none) -> picowalker:SIT1533AIH4DCC32768E
Changed lines of the file:
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@@
 			)
 		)
-		(property "Footprint" ""
+		(property "Footprint" "picowalker:SIT1533AIH4DCC32768E"
 			(at 139.7 153.34 0)
 			(effects

Commit message: v0.4: drc mostly done, need to fiddle with TH1
Parts:
- added TP3: 32k, picowalker:TestPoint_Pad_D1.0mm_Nosilk, symbol Connector:TestPoint
- added TP4: GND, picowalker:TestPoint_Pad_D1.0mm_Nosilk, symbol Connector:TestPoint
Connections:
- net CLK: now also TP3.1
- net GND: now also TP4.1
Other:
- note added: "32768 Hz 75 ppm stability from -10 C to +70 C 20 ppm tolerance 1 ppm aging (1 year) = ~100 ppm = +/-4 Hz = ~ 9 seconds/day max drift"
Changed lines of the file:
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@@
 	(generator_version "9.0")
 	(paper "A4")
-	(wire
-		(pts
-			(xy 128.27 81.28) (xy 128.27 86.36)
+	(text "32768 Hz\n75 ppm stability from -10 C to +70 C\n20 ppm tolerance\n1 ppm aging (1 year)\n\n= ~100 ppm = +/-4 Hz\n= ~ 9 seconds/day max drift"
+		(exclude_from_sim no)
+		(at 142.24 36.322 0)
+		(effects
+			(font
+				(size 1.27 1.27)
+			)
+			(justify left top)
+		)
+	)
+	(junction
+		(at 151.13 66.04)
+		(diameter 0)
+		(color 0 0 0 0)
+	)
+	(junction
+		(at 128.27 83.82)
+		(diameter 0)
+		(color 0 0 0 0)
+	)
+	(wire
+		(pts
+			(xy 128.27 81.28) (xy 128.27 83.82)
 		)
 		(stroke
@@
 	(wire
 		(pts
-			(xy 143.51 66.04) (xy 149.86 66.04)
+			(xy 132.08 83.82) (xy 128.27 83.82)
+		)
+		(stroke
+			(width 0)
+			(type default)
+		)
+	)
+	(wire
+		(pts
+			(xy 143.51 66.04) (xy 151.13 66.04)
+		)
+		(stroke
+			(width 0)
+			(type default)
+		)
+	)
+	(wire
+		(pts
+			(xy 151.13 66.04) (xy 167.64 66.04)
+		)
+		(stroke
+			(width 0)
+			(type default)
+		)
+	)
+	(wire
+		(pts
+			(xy 128.27 83.82) (xy 128.27 86.36)
 		)
 		(stroke
@@
 	(hierarchical_label "CLK"
 		(shape output)
-		(at 149.86 66.04 0)
+		(at 167.64 66.04 0)
 		(effects
 			(font
@@
 		(on_board yes)
 		(dnp no)
-		(fields_autoplaced yes)
 		(property "Reference" "Y2"
-			(at 153.67 59.6198 0)
+			(at 108.204 51.054 0)
 			(effects
 				(font
@@
 		)
 		(property "Value" "SIT1533AI-H4-DCC-32.768E"
-			(at 153.67 62.1598 0)
+			(at 108.204 53.594 0)
 			(effects
 				(font
@@
 				(path "/aa8773bf-a88b-4bf9-9961-8e312cd9d0e3/feaa0ed6-677d-464b-a267-7ec72771ce12"
 					(reference "Y2")
+					(unit 1)
+				)
+			)
+		)
+	)
+	(symbol
+		(lib_id "Connector:TestPoint")
+		(at 132.08 83.82 0)
+		(unit 1)
+		(exclude_from_sim no)
+		(in_bom yes)
+		(on_board yes)
+		(dnp no)
+		(fields_autoplaced yes)
+		(property "Reference" "TP4"
+			(at 134.62 79.2479 0)
+			(effects
+				(font
+					(size 1.27 1.27)
+				)
+				(justify left)
+			)
+		)
+		(property "Value" "GND"
+			(at 134.62 81.7879 0)
+			(effects
+				(font
+					(size 1.27 1.27)
+				)
+				(justify left)
+			)
+		)
+		(property "Footprint" "picowalker:TestPoint_Pad_D1.0mm_Nosilk"
+			(at 137.16 83.82 0)
+			(effects
+				(font
+					(size 1.27 1.27)
+				)
+				(hide yes)
+			)
+		)
+		(property "Datasheet" "~"
+			(at 137.16 83.82 0)
+			(effects
+				(font
+					(size 1.27 1.27)
+				)
+				(hide yes)
+			)
+		)
+		(property "Description" "test point"
+			(at 132.08 83.82 0)
+			(effects
+				(font
+					(size 1.27 1.27)
+				)
+				(hide yes)
+			)
+		)
+		(pin "1"
+		)
+		(instances
+			(project "picowalker-v0.4"
+				(path "/aa8773bf-a88b-4bf9-9961-8e312cd9d0e3/feaa0ed6-677d-464b-a267-7ec72771ce12"
+					(reference "TP4")
 					(unit 1)
 				)
@@
 					(unit 1)
 				)
+			)
+		)
+	)
+	(symbol
+		(lib_id "Connector:TestPoint")
+		(at 151.13 66.04 0)
+		(unit 1)
+		(exclude_from_sim no)
+		(in_bom yes)
+		(on_board yes)
+		(dnp no)
+		(fields_autoplaced yes)
+		(property "Reference" "TP3"
+			(at 153.67 61.4679 0)
+			(effects
+				(font
+					(size 1.27 1.27)
+				)
+				(justify left)
+			)
+		)
+		(property "Value" "32k"
+			(at 153.67 64.0079 0)
+			(effects
+				(font
+					(size 1.27 1.27)
+				)
+				(justify left)
+			)
+		)
+		(property "Footprint" "picowalker:TestPoint_Pad_D1.0mm_Nosilk"
+			(at 156.21 66.04 0)
+			(effects
+				(font
+					(size 1.27 1.27)
+				)
+				(hide yes)
+			)
+		)
+		(property "Datasheet" "~"
+			(at 156.21 66.04 0)
+			(effects
+				(font
+					(size 1.27 1.27)
+				)
+				(hide yes)
+			)
+		)
+		(property "Description" "test point"
+			(at 151.13 66.04 0)
+			(effects
+				(font
+					(size 1.27 1.27)
+				)
+				(hide yes)
+			)
+		)
+		(pin "1"
+		)
+		(instances
+			(project ""
+				(path "/aa8773bf-a88b-4bf9-9961-8e312cd9d0e3/feaa0ed6-677d-464b-a267-7ec72771ce12"
+					(reference "TP3")
+					(unit 1)
+				)

Commit message: v0.4: idk, minimal changes
Parts:
- TP3, TP4: now left out of the parts list
Changed lines of the file:
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@@
 		(unit 1)
 		(exclude_from_sim no)
-		(in_bom yes)
+		(in_bom no)
 		(on_board yes)
 		(dnp no)
@@
 		(unit 1)
 		(exclude_from_sim no)
-		(in_bom yes)
+		(in_bom no)
 		(on_board yes)
 		(dnp no)
